File: Designs/Autopilot Control Unit rev2.brd (EAGLE design)
At the start: 59.9 x 37.3 mm, 43 parts, among them J1 CONNECTOR_3__0.1"_INCH_TH, J10 CONNECTOR_3__0.1"_INCH_TH, J11 CONNECTOR_3__0.1"_INCH_TH, J12 CONNECTOR_3__0.1"_INCH_TH, J2 CONNECTOR_3__0.1"_INCH_TH, J3 CONNECTOR_3__0.1"_INCH_TH, J4 CONNECTOR_3__0.1"_INCH_TH, J5 CONNECTOR_3__0.1"_INCH_TH, J6 CONNECTOR_3__0.1"_INCH_TH, J7 CONNECTOR_3__0.1"_INCH_TH, J8 CONNECTOR_3__0.1"_INCH_TH, J9 CONNECTOR_3__0.1"_INCH_TH, U1 ICM-42605, U2 VOLTAGE_REGULATOR_SOT-23-5_5V, U3 ADG1421, U4 ADG1421, U5 ADG1421

Commit message: rev2
Parts:
- removed R13, R14, R15, R16, R17, R18: RESISTOR_0603_10K, HyTechDevices:0603-RES
- removed U3, U4, U5: ADG1421, Devices:MSOP-10
- R10, R12, R2, R4, R6, R8: value RESISTOR_0603_10K -> RESISTOR_0603_15K
Connections:
- removed net AILERON_OUT: J9.2, R14.2, U3.9
- removed net AUX_OUT: J7.2, R18.2, U5.9
- removed net ELEVATOR_OUT: J10.2, R15.2, U4.10
- removed net GEAR_OUT: J12.2, R17.2, U5.10
- removed net RUDDER_OUT: J11.2, R16.2, U4.9
- removed net THROTTLE_OUT: J8.2, R13.2, U3.10
- net AILERON_CTRL: now also J9.2; no longer U3.6
- net AUX_CTRL: now also J7.2; no longer U5.6
- net ELEVATOR_CTRL: now also J10.2; no longer U4.7
- net GEAR_CTRL: now also J12.2; no longer U5.7
- net GND: no longer R13.1, R14.1, R15.1, R16.1, R17.1, R18.1, U3.4, U3.8, U4.4, U4.8, U5.4, U5.8
- net RUDDER_CTRL: now also J11.2; no longer U4.6
- net THROTTLE_CTRL: now also J8.2; no longer U3.7
- net VBAT: no longer U3.1, U3.2, U3.5, U4.1, U4.2, U4.5, U5.1, U5.2, U5.5
Routing:
- net VBAT: track 145.1 -> 105.7 mm
- net RUDDER_OUT: track 28.2 -> 0.00 mm
- net GND: track 46.7 -> 21.8 mm, vias 21 -> 13
- net ELEVATOR_OUT: track 21.1 -> 0.00 mm
- net AILERON_OUT: track 18.8 -> 0.00 mm
- net GEAR_OUT: track 14.6 -> 0.00 mm
- net AUX_OUT: track 12.4 -> 0.00 mm
- net RUDDER_CTRL: track 62.9 -> 50.9 mm
- net AILERON_CTRL: track 29.2 -> 41.1 mm
- net THROTTLE_OUT: track 11.8 -> 0.00 mm
- net GEAR_CTRL: track 29.9 -> 39.4 mm
- net ELEVATOR_CTRL: track 53.2 -> 44.8 mm
- net AUX_CTRL: track 32.6 -> 39.2 mm
- net THROTTLE_CTRL: track 29.2 -> 32.6 mm
Other:
- board size 59.9 x 37.3 mm -> 57.9 x 37.3 mm
- board text added: "Autopilot Control Unit Rev2 Zekun Li"
- board text removed: "Autopilot Control Unit Rev1 Zekun Li"
