File: Designs/Autopilot Control Unit rev2.sch (EAGLE design)
At the start: 44 parts, among them J1 CONNECTOR_3__0.1"_INCH_TH, J10 CONNECTOR_3__0.1"_INCH_TH, J11 CONNECTOR_3__0.1"_INCH_TH, J12 CONNECTOR_3__0.1"_INCH_TH, J2 CONNECTOR_3__0.1"_INCH_TH, J3 CONNECTOR_3__0.1"_INCH_TH, J4 CONNECTOR_3__0.1"_INCH_TH, J5 CONNECTOR_3__0.1"_INCH_TH, J6 CONNECTOR_3__0.1"_INCH_TH, J7 CONNECTOR_3__0.1"_INCH_TH, J8 CONNECTOR_3__0.1"_INCH_TH, J9 CONNECTOR_3__0.1"_INCH_TH, Q1 TRANSISTOR_N_MOS__PMV15ENEA, Q2 TRANSISTOR_N_MOS__PMV15ENEA, Q3 TRANSISTOR_N_MOS__PMV15ENEA, Q4 TRANSISTOR_N_MOS__PMV15ENEA, Q5 TRANSISTOR_N_MOS__PMV15ENEA, Q6 TRANSISTOR_N_MOS__PMV15ENEA, U1 ICM-42605, U2 VOLTAGE_REGULATOR_SOT-23-5_5V

Commit message: rev2
Parts:
- removed Q1, Q2, Q3, Q4, Q5, Q6: TRANSISTOR_N_MOS__PMV15ENEA, HyTechDevices:TRANSISTOR_N_MOS__PMV15ENEA
- removed R13, R14, R15, R16, R17, R18: RESISTOR_0603_10K, HyTechDevices:RESISTOR_0603_10K
- R10, R12, R2, R4, R6, R8: value RESISTOR_0603_10K -> RESISTOR_0603_15K; device HyTechDevices:RESISTOR_0603_10K -> HyTechDevices:RESISTOR_0603_15K
Connections:
- removed net AILERON_OUT: J9.2, Q2.S, R17.2
- removed net AUX_OUT: J7.2, Q6.S, R15.2
- removed net ELEVATOR_OUT: J10.2, Q3.S, R18.2
- removed net GEAR_OUT: J12.2, Q5.S, R14.2
- removed net RUDDER_OUT: J11.2, Q4.S, R13.2
- removed net THROTTLE_OUT: J8.2, Q1.S, R16.2
- net AILERON_CTRL: now also J9.2; no longer Q2.G
- net AUX_CTRL: now also J7.2; no longer Q6.G
- net ELEVATOR_CTRL: now also J10.2; no longer Q3.G
- net GEAR_CTRL: now also J12.2; no longer Q5.G
- net GND: no longer R13.1, R14.1, R15.1, R16.1, R17.1, R18.1
- net RUDDER_CTRL: now also J11.2; no longer Q4.G
- net THROTTLE_CTRL: now also J8.2; no longer Q1.G
- net VBAT: no longer Q1.D, Q2.D, Q3.D, Q4.D, Q5.D, Q6.D
Other:
- moved on the sheet: J10, J11, J12, J7, J8, J9
